Commit message: clar02_husky.urdf.xacro edited online with Bitbucket

File: urdf/clar02_husky.urdf.xacro (robot description, xacro)
@@ -6,5 +6,5 @@
     <parent link="base_link"/>
     <child link="laser"/>
-    <origin xyz="0.29220145206 0.0 0.44619757154" rpy="$0.0 0.0 0.0"/>
+    <origin xyz="0.29220145206 0.0 0.44619757154" rpy="0.0 0.0 0.0"/>
   </joint>
   <link name="laser" />

Commit message: Modified the xacro file and added sick launcher

File: urdf/clar02_husky.urdf.xacro (robot description, xacro)
@@ -6,5 +6,5 @@
     <parent link="base_link"/>
     <child link="laser"/>
-    <origin xyz="0.29220145206 0.0 0.44619757154" rpy="0.0 0.0 0.0"/>
+    <origin xyz="0.29220145206 0.0 0.44619757154" rpy="3.14159 0.0 0.0"/>
   </joint>
   <link name="laser" />
